Commit message: slam funct with hickups

File: travis_description/urdf/travis.xacro (robot description, xacro)
@@ -6,5 +6,5 @@
 <link name="robot_footprint"></link>
   <joint name="robot_footprint_joint" type="fixed">
-    <origin xyz="0 0 0" rpy="0 0 0" />
+    <origin xyz="0 0 0" rpy="0 0 3.1415" />
     <parent link="robot_footprint" />
     <child link="base_link" />

Commit message: switched around lidar and cmdvelx

File: travis_description/urdf/travis.xacro (robot description, xacro)
@@ -480,5 +480,5 @@
 </joint>
 <joint name="Rigid24" type="fixed">
-  <origin xyz="-0.0455 0.0 0.041512" rpy="0 0 0"/>
+  <origin xyz="-0.0455 0.0 0.041512" rpy="0 0 3.1415"/>
   <parent link="rp_lidar_base_1"/>
   <child link="lidar_1"/>
